Commit message: change position

File: tankbot_description/urdf/tankbot.xacro (robot description, xacro)
@@ -6,7 +6,7 @@
 <link name="base_link">
   <inertial>
-    <origin xyz="0.04802449670948884 -0.2570000000000001 0.03092345572753796" rpy="0 0 0"/>
-    <mass value="9.663393854812522"/>
-    <inertia ixx="0.050312" iyy="0.087124" izz="0.121613" ixy="-0.0" iyz="-0.0" ixz="-1.3e-05"/>
+    <origin xyz="-0.0019755032905111897 -0.007000000000000141 0.030923455727537946" rpy="0 0 0"/>
+    <mass value="9.66339385481253"/>
+    <inertia ixx="0.050312" iyy="0.087124" izz="0.121613" ixy="-0.0" iyz="0.0" ixz="-1.3e-05"/>
   </inertial>
   <visual>
@@ -24,72 +24,112 @@
   </collision>
 </link>
+<link name="rw1_link_1">
+  <inertial>
+    <origin xyz="-2.914335439641036e-16 -0.015000000000000083 -7.632783294297951e-17" rpy="0 0 0"/>
+    <mass value="1.6692754390078937"/>
+    <inertia ixx="0.001067" iyy="0.001883" izz="0.001067" ixy="0.0" iyz="0.0" ixz="-0.0"/>
+  </inertial>
+  <visual>
+    <origin xyz="-0.1 0.1135 -0.035" rpy="0 0 0"/>
+    <geometry>
+      <mesh filename="package://tankbot_description/meshes/rw1_link_1.stl" scale="0.001 0.001 0.001"/>
+    </geometry>
+    <material name="silver"/>
+  </visual>
+  <collision>
+    <origin xyz="-0.1 0.1135 -0.035" rpy="0 0 0"/>
+    <geometry>
+      <mesh filename="package://tankbot_description/meshes/rw1_link_1.stl" scale="0.001 0.001 0.001"/>
+    </geometry>
+  </collision>
+</link>
+<link name="rw2_link_1">
+  <inertial>
+    <origin xyz="1.5612511283791264e-17 -0.01500000000000025 1.1102230246251565e-16" rpy="0 0 0"/>
+    <mass value="1.6692754390078943"/>
+    <inertia ixx="0.001067" iyy="0.001883" izz="0.001067" ixy="0.0" iyz="-0.0" ixz="-0.0"/>
+  </inertial>
+  <visual>
+    <origin xyz="0.0025 0.1135 -0.035" rpy="0 0 0"/>
+    <geometry>
+      <mesh filename="package://tankbot_description/meshes/rw2_link_1.stl" scale="0.001 0.001 0.001"/>
+    </geometry>
+    <material name="silver"/>
+  </visual>
+  <collision>
+    <origin xyz="0.0025 0.1135 -0.035" rpy="0 0 0"/>
+    <geometry>
+      <mesh filename="package://tankbot_description/meshes/rw2_link_1.stl" scale="0.001 0.001 0.001"/>
+    </geometry>
+  </collision>
+</link>
 <link name="rw3_link_1">
   <inertial>
-    <origin xyz="-2.7755575615628914e-17 -0.015000000000000069 -2.0816681711721685e-17" rpy="0 0 0"/>
-    <mass value="1.6692754390078943"/>
+    <origin xyz="-6.938893903907228e-17 -0.01500000000000011 -4.163336342344337e-17" rpy="0 0 0"/>
+    <mass value="1.6692754390078937"/>
+    <inertia ixx="0.001067" iyy="0.001883" izz="0.001067" ixy="-0.0" iyz="0.0" ixz="0.0"/>
+  </inertial>
+  <visual>
+    <origin xyz="0.105 0.1135 -0.035" rpy="0 0 0"/>
+    <geometry>
+      <mesh filename="package://tankbot_description/meshes/rw3_link_1.stl" scale="0.001 0.001 0.001"/>
+    </geometry>
+    <material name="silver"/>
+  </visual>
+  <collision>
+    <origin xyz="0.105 0.1135 -0.035" rpy="0 0 0"/>
+    <geometry>
+      <mesh filename="package://tankbot_description/meshes/rw3_link_1.stl" scale="0.001 0.001 0.001"/>
+    </geometry>
+  </collision>
+</link>
+<link name="lw3_link_1">
+  <inertial>
+    <origin xyz="1.249000902703301e-16 0.014999999999999958 6.938893903907228e-18" rpy="0 0 0"/>
+    <mass value="1.6692754390078937"/>
+    <inertia ixx="0.001067" iyy="0.001883" izz="0.001067" ixy="-0.0" iyz="0.0" ixz="0.0"/>
+  </inertial>
+  <visual>
+    <origin xyz="0.1045 -0.0995 -0.035" rpy="0 0 0"/>
+    <geometry>
+      <mesh filename="package://tankbot_description/meshes/lw3_link_1.stl" scale="0.001 0.001 0.001"/>
+    </geometry>
+    <material name="silver"/>
+  </visual>
+  <collision>
+    <origin xyz="0.1045 -0.0995 -0.035" rpy="0 0 0"/>
+    <geometry>
+      <mesh filename="package://tankbot_description/meshes/lw3_link_1.stl" scale="0.001 0.001 0.001"/>
+    </geometry>
+  </collision>
+</link>
+<link name="lw2_link_1">
+  <inertial>
+    <origin xyz="4.206704429243757e-17 0.014999999999999986 -2.7755575615628914e-17" rpy="0 0 0"/>
+    <mass value="1.6692754390078937"/>
+    <inertia ixx="0.001067" iyy="0.001883" izz="0.001067" ixy="-0.0" iyz="-0.0" ixz="0.0"/>
+  </inertial>
+  <visual>
+    <origin xyz="0.002 -0.0995 -0.035" rpy="0 0 0"/>
+    <geometry>
+      <mesh filename="package://tankbot_description/meshes/lw2_link_1.stl" scale="0.001 0.001 0.001"/>
+    </geometry>
+    <material name="silver"/>
+  </visual>
+  <collision>
+    <origin xyz="0.002 -0.0995 -0.035" rpy="0 0 0"/>
+    <geometry>
+      <mesh filename="package://tankbot_description/meshes/lw2_link_1.stl" scale="0.001 0.001 0.001"/>
+    </geometry>
+  </collision>
+</link>
+<link name="lw1_link_1">
+  <inertial>
+    <origin xyz="4.163336342344337e-17 0.014999999999999986 -9.020562075079397e-17" rpy="0 0 0"/>
+    <mass value="1.6692754390078937"/>
     <inertia ixx="0.001067" iyy="0.001883" izz="0.001067" ixy="0.0" iyz="0.0" ixz="0.0"/>
   </inertial>
   <visual>
-    <origin xyz="0.055 0.3635 -0.035" rpy="0 0 0"/>
-    <geometry>
-      <mesh filename="package://tankbot_description/meshes/rw3_link_1.stl" scale="0.001 0.001 0.001"/>
-    </geometry>
-    <material name="silver"/>
-  </visual>
-  <collision>
-    <origin xyz="0.055 0.3635 -0.035" rpy="0 0 0"/>
-    <geometry>
-      <mesh filename="package://tankbot_description/meshes/rw3_link_1.stl" scale="0.001 0.001 0.001"/>
-    </geometry>
-  </collision>
-</link>
-<link name="rw2_link_1">
-  <inertial>
-    <origin xyz="2.7755575615628914e-17 -0.015000000000000513 9.020562075079397e-17" rpy="0 0 0"/>
-    <mass value="1.669275439007894"/>
-    <inertia ixx="0.001067" iyy="0.001883" izz="0.001067" ixy="-0.0" iyz="-0.0" ixz="-0.0"/>
-  </inertial>
-  <visual>
-    <origin xyz="-0.0475 0.3635 -0.035" rpy="0 0 0"/>
-    <geometry>
-      <mesh filename="package://tankbot_description/meshes/rw2_link_1.stl" scale="0.001 0.001 0.001"/>
-    </geometry>
-    <material name="silver"/>
-  </visual>
-  <collision>
-    <origin xyz="-0.0475 0.3635 -0.035" rpy="0 0 0"/>
-    <geometry>
-      <mesh filename="package://tankbot_description/meshes/rw2_link_1.stl" scale="0.001 0.001 0.001"/>
-    </geometry>
-  </collision>
-</link>
-<link name="rw1_link_1">
-  <inertial>
-    <origin xyz="-1.1102230246251565e-16 -0.015000000000000013 1.3877787807814457e-17" rpy="0 0 0"/>
-    <mass value="1.6692754390078939"/>
-    <inertia ixx="0.001067" iyy="0.001883" izz="0.001067" ixy="0.0" iyz="-0.0" ixz="-0.0"/>
-  </inertial>
-  <visual>
-    <origin xyz="-0.15 0.3635 -0.035" rpy="0 0 0"/>
-    <geometry>
-      <mesh filename="package://tankbot_description/meshes/rw1_link_1.stl" scale="0.001 0.001 0.001"/>
-    </geometry>
-    <material name="silver"/>
-  </visual>
-  <collision>
-    <origin xyz="-0.15 0.3635 -0.035" rpy="0 0 0"/>
-    <geometry>
-      <mesh filename="package://tankbot_description/meshes/rw1_link_1.stl" scale="0.001 0.001 0.001"/>
-    </geometry>
-  </collision>
-</link>
-<link name="lw1_link_1">
-  <inertial>
-    <origin xyz="1.1102230246251565e-16 0.014999999999999902 3.469446951953614e-17" rpy="0 0 0"/>
-    <mass value="1.6692754390078937"/>
-    <inertia ixx="0.001067" iyy="0.001883" izz="0.001067" ixy="0.0" iyz="0.0" ixz="0.0"/>
-  </inertial>
-  <visual>
-    <origin xyz="-0.1505 0.1505 -0.035" rpy="0 0 0"/>
+    <origin xyz="-0.1005 -0.0995 -0.035" rpy="0 0 0"/>
     <geometry>
       <mesh filename="package://tankbot_description/meshes/lw1_link_1.stl" scale="0.001 0.001 0.001"/>
@@ -98,5 +138,5 @@
   </visual>
   <collision>
-    <origin xyz="-0.1505 0.1505 -0.035" rpy="0 0 0"/>
+    <origin xyz="-0.1005 -0.0995 -0.035" rpy="0 0 0"/>
     <geometry>
       <mesh filename="package://tankbot_description/meshes/lw1_link_1.stl" scale="0.001 0.001 0.001"/>
@@ -104,52 +144,12 @@
   </collision>
 </link>
-<link name="lw2_link_1">
-  <inertial>
-    <origin xyz="6.245004513516506e-17 0.014999999999999875 2.7755575615628914e-17" rpy="0 0 0"/>
-    <mass value="1.6692754390078937"/>
-    <inertia ixx="0.001067" iyy="0.001883" izz="0.001067" ixy="0.0" iyz="0.0" ixz="0.0"/>
-  </inertial>
-  <visual>
-    <origin xyz="-0.048 0.1505 -0.035" rpy="0 0 0"/>
-    <geometry>
-      <mesh filename="package://tankbot_description/meshes/lw2_link_1.stl" scale="0.001 0.001 0.001"/>
-    </geometry>
-    <material name="silver"/>
-  </visual>
-  <collision>
-    <origin xyz="-0.048 0.1505 -0.035" rpy="0 0 0"/>
-    <geometry>
-      <mesh filename="package://tankbot_description/meshes/lw2_link_1.stl" scale="0.001 0.001 0.001"/>
-    </geometry>
-  </collision>
-</link>
-<link name="lw3_link_1">
-  <inertial>
-    <origin xyz="9.71445146547012e-17 0.01499999999999993 2.7755575615628914e-17" rpy="0 0 0"/>
-    <mass value="1.6692754390078937"/>
-    <inertia ixx="0.001067" iyy="0.001883" izz="0.001067" ixy="0.0" iyz="0.0" ixz="0.0"/>
-  </inertial>
-  <visual>
-    <origin xyz="0.0545 0.1505 -0.035" rpy="0 0 0"/>
-    <geometry>
-      <mesh filename="package://tankbot_description/meshes/lw3_link_1.stl" scale="0.001 0.001 0.001"/>
-    </geometry>
-    <material name="silver"/>
-  </visual>
-  <collision>
-    <origin xyz="0.0545 0.1505 -0.035" rpy="0 0 0"/>
-    <geometry>
-      <mesh filename="package://tankbot_description/meshes/lw3_link_1.stl" scale="0.001 0.001 0.001"/>
-    </geometry>
-  </collision>
-</link>
 <link name="frame_1">
   <inertial>
-    <origin xyz="1.1856979425378666e-07 -1.1102230246251565e-16 0.1270000000000003" rpy="0 0 0"/>
-    <mass value="4.173751809755388"/>
-    <inertia ixx="0.053156" iyy="0.059602" izz="0.047225" ixy="0.0" iyz="0.0" ixz="0.0"/>
-  </inertial>
-  <visual>
-    <origin xyz="-0.048432 0.2575 -0.09" rpy="0 0 0"/>
+    <origin xyz="9.410874857174178e-17 -3.382710778154774e-17 0.12700000000000053" rpy="0 0 0"/>
+    <mass value="4.173751809755377"/>
+    <inertia ixx="0.053156" iyy="0.059602" izz="0.047225" ixy="-0.0" iyz="0.0" ixz="0.0"/>
+  </inertial>
+  <visual>
+    <origin xyz="0.002 0.007 -0.09" rpy="0 0 0"/>
     <geometry>
       <mesh filename="package://tankbot_description/meshes/frame_1.stl" scale="0.001 0.001 0.001"/>
@@ -158,5 +158,5 @@
   </visual>
   <collision>
-    <origin xyz="-0.048432 0.2575 -0.09" rpy="0 0 0"/>
+    <origin xyz="0.002 0.007 -0.09" rpy="0 0 0"/>
     <geometry>
       <mesh filename="package://tankbot_description/meshes/frame_1.stl" scale="0.001 0.001 0.001"/>
@@ -166,10 +166,10 @@
 <link name="holder_1">
   <inertial>
-    <origin xyz="-0.015898641976588364 -0.0001410013794365672 0.03722253654962837" rpy="0 0 0"/>
+    <origin xyz="-0.015898760546382822 -0.0001410013794365464 0.037222536549628205" rpy="0 0 0"/>
     <mass value="2.1421450013668144"/>
     <inertia ixx="0.010373" iyy="0.004839" izz="0.011427" ixy="1.1e-05" iyz="-5e-06" ixz="6.3e-05"/>
   </inertial>
   <visual>
-    <origin xyz="-0.048432 0.2575 -0.344" rpy="0 0 0"/>
+    <origin xyz="-0.018 0.007 -0.344" rpy="0 0 0"/>
     <geometry>
       <mesh filename="package://tankbot_description/meshes/holder_1.stl" scale="0.001 0.001 0.001"/>
@@ -178,5 +178,5 @@
   </visual>
   <collision>
-    <origin xyz="-0.048432 0.2575 -0.344" rpy="0 0 0"/>
+    <origin xyz="-0.018 0.007 -0.344" rpy="0 0 0"/>
     <geometry>
       <mesh filename="package://tankbot_description/meshes/holder_1.stl" scale="0.001 0.001 0.001"/>
@@ -186,10 +186,10 @@
 <link name="camera_1">
   <inertial>
-    <origin xyz="0.005000020162195945 1.3403930410049725e-07 1.1102230246251565e-16" rpy="0 0 0"/>
+    <origin xyz="0.004999901592401532 1.3403930415253895e-07 5.551115123125783e-17" rpy="0 0 0"/>
     <mass value="0.15204665638341558"/>
-    <inertia ixx="0.000106" iyy="7e-06" izz="0.000102" ixy="-0.0" iyz="0.0" ixz="-0.0"/>
-  </inertial>
-  <visual>
-    <origin xyz="-0.072341 0.260428 -0.367" rpy="0 0 0"/>
+    <inertia ixx="0.000106" iyy="7e-06" izz="0.000102" ixy="0.0" iyz="-0.0" ixz="0.0"/>
+  </inertial>
+  <visual>
+    <origin xyz="-0.041909 0.009928 -0.367" rpy="0 0 0"/>
     <geometry>
       <mesh filename="package://tankbot_description/meshes/camera_1.stl" scale="0.001 0.001 0.001"/>
@@ -198,5 +198,5 @@
   </visual>
   <collision>
-    <origin xyz="-0.072341 0.260428 -0.367" rpy="0 0 0"/>
+    <origin xyz="-0.041909 0.009928 -0.367" rpy="0 0 0"/>
     <geometry>
       <mesh filename="package://tankbot_description/meshes/camera_1.stl" scale="0.001 0.001 0.001"/>
@@ -206,10 +206,10 @@
 <link name="lidar_1">
   <inertial>
-    <origin xyz="-4.29900122521365e-07 -2.5480986765025193e-09 0.019135896206633696" rpy="0 0 0"/>
-    <mass value="1.898390048800237"/>
+    <origin xyz="4.515300830107427e-07 -2.5480985724191108e-09 0.019135896206633585" rpy="0 0 0"/>
+    <mass value="1.8983900488002365"/>
     <inertia ixx="0.001161" iyy="0.001161" izz="0.001848" ixy="0.0" iyz="-0.0" ixz="-0.0"/>
   </inertial>
   <visual>
-    <origin xyz="-0.048387 0.2575 -0.42" rpy="0 0 0"/>
+    <origin xyz="-0.017954 0.007 -0.42" rpy="0 0 0"/>
     <geometry>
       <mesh filename="package://tankbot_description/meshes/lidar_1.stl" scale="0.001 0.001 0.001"/>
@@ -218,5 +218,5 @@
   </visual>
   <collision>
-    <origin xyz="-0.048387 0.2575 -0.42" rpy="0 0 0"/>
+    <origin xyz="-0.017954 0.007 -0.42" rpy="0 0 0"/>
     <geometry>
       <mesh filename="package://tankbot_description/meshes/lidar_1.stl" scale="0.001 0.001 0.001"/>
@@ -224,47 +224,47 @@
   </collision>
 </link>
+<joint name="rw1_joint" type="continuous">
+  <origin xyz="0.1 -0.1135 0.035" rpy="0 0 0"/>
+  <parent link="base_link"/>
+  <child link="rw1_link_1"/>
+  <axis xyz="-0.0 1.0 0.0"/>
+</joint>
+<joint name="rw2_joint" type="continuous">
+  <origin xyz="-0.0025 -0.1135 0.035" rpy="0 0 0"/>
+  <parent link="base_link"/>
+  <child link="rw2_link_1"/>
+  <axis xyz="-0.0 1.0 0.0"/>
+</joint>
 <joint name="rw3_joint" type="continuous">
-  <origin xyz="-0.055 -0.3635 0.035" rpy="0 0 0"/>
+  <origin xyz="-0.105 -0.1135 0.035" rpy="0 0 0"/>
   <parent link="base_link"/>
   <child link="rw3_link_1"/>
   <axis xyz="-0.0 1.0 0.0"/>
 </joint>
-<joint name="rw2_joint" type="continuous">
-  <origin xyz="0.0475 -0.3635 0.035" rpy="0 0 0"/>
-  <parent link="base_link"/>
-  <child link="rw2_link_1"/>
-  <axis xyz="-0.0 1.0 0.0"/>
-</joint>
-<joint name="rw1_joint" type="continuous">
-  <origin xyz="0.15 -0.3635 0.035" rpy="0 0 0"/>
-  <parent link="base_link"/>
-  <child link="rw1_link_1"/>
-  <axis xyz="-0.0 1.0 0.0"/>
+<joint name="lw3_joint" type="continuous">
+  <origin xyz="-0.1045 0.0995 0.035" rpy="0 0 0"/>
+  <parent link="base_link"/>
+  <child link="lw3_link_1"/>
+  <axis xyz="0.0 1.0 0.0"/>
+</joint>
+<joint name="lw2_joint" type="continuous">
+  <origin xyz="-0.002 0.0995 0.035" rpy="0 0 0"/>
+  <parent link="base_link"/>
+  <child link="lw2_link_1"/>
+  <axis xyz="0.0 1.0 0.0"/>
 </joint>
 <joint name="lw1_joint" type="continuous">
-  <origin xyz="0.1505 -0.1505 0.035" rpy="0 0 0"/>
+  <origin xyz="0.1005 0.0995 0.035" rpy="0 0 0"/>
   <parent link="base_link"/>
   <child link="lw1_link_1"/>
   <axis xyz="0.0 1.0 0.0"/>
 </joint>
-<joint name="lw2_joint" type="continuous">
-  <origin xyz="0.048 -0.1505 0.035" rpy="0 0 0"/>
-  <parent link="base_link"/>
-  <child link="lw2_link_1"/>
-  <axis xyz="0.0 1.0 0.0"/>
-</joint>
-<joint name="lw3_joint" type="continuous">
-  <origin xyz="-0.0545 -0.1505 0.035" rpy="0 0 0"/>
-  <parent link="base_link"/>
-  <child link="lw3_link_1"/>
-  <axis xyz="0.0 1.0 0.0"/>
-</joint>
 <joint name="frame_joint" type="fixed">
-  <origin xyz="0.048432 -0.2575 0.09" rpy="0 0 0"/>
+  <origin xyz="-0.002 -0.007 0.09" rpy="0 0 0"/>
   <parent link="base_link"/>
   <child link="frame_1"/>
 </joint>
 <joint name="holder_joint" type="fixed">
-  <origin xyz="0.0 0.0 0.254" rpy="0 0 0"/>
+  <origin xyz="0.02 0.0 0.254" rpy="0 0 0"/>
   <parent link="frame_1"/>
   <child link="holder_1"/>
@@ -276,5 +276,5 @@
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